File: Hand_solder/USB_C_PD_Prototyping_Board_hand_solder.kicad_sch (KiCad schematic)
At the start: 48 parts, among them IC1 TPS259474LRPWR, J1 USB_C_Receptacle, J2 Power_out, J3 Data_out, J5 Conn_01x04_Pin, J6 Conn_02x02_Counter_Clockwise, J7 Conn_02x02_Counter_Clockwise, Q1 DMP3018SFV-7, Q2 DMP3018SFV-7, SW1 Power_out_switch, U1 HUSB238_xxxDD, U2 K7803-500R3_C909766

Commit message: Seperate hand solder and ready to use versions
Parts:
- R1, R10, R11, R12, R14, R15, R16, R17, R2, R20, R21, R3, R4, R5, R7, R8, R9: footprint Resistor_SMD:R_0402_1005Metric_Pad0.72x0.64mm_HandSolder -> Resistor_THT:R_Axial_DIN0207_L6.3mm_D2.5mm_P7.62mm_Horizontal
